File: BoBa/BoBa.kicad_pcb (KiCad board)
At the start: 4 copper layers, 90.3 x 95.8 mm, 41 parts, among them J1 DF13C-2P-1.25V(21), J2 DF13C-2P-1.25V(21), J3 DF13C-2P-1.25V(21), J4 DF13C-2P-1.25V(21), Q1 FQD13N06LTM, Q2 FQD13N06LTM, U1 LTC4231HUD-2#TRPBF, U2 INA219, U3 INA219AIDCNR, U4_IN-A LTC4231IUD-2#TRPBF, U5 INA219AIDCNR

Commit message: Update BoBa.kicad_pcb
Routing:
- net NetQ2_1: track 68.9 -> 58.7 mm
Changed lines of the file:
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@@
 		)
 	)
+	(property "SHEETTOTAL" "3")
 	(footprint "SnapEDA_Library:SAMTEC_SSQ-126-X-G-D"
 		(layer "F.Cu")
@@
 	)
 	(segment
-		(start 165.68314 94.48452)
-		(end 167.65544 94.48452)
-		(width 0.2)
-		(layer "B.Cu")
-		(net "NetQ2_1")
-	)
-	(segment
 		(start 170.4713 110.10982)
 		(end 175.74114 104.83998)
@@
 	)
 	(segment
-		(start 168.19049 92.44947)
-		(end 168.19049 89.04547)
-		(width 0.254)
-		(layer "B.Cu")
-		(net "NetQ2_1")
-	)
-	(segment
-		(start 168.19049 89.04547)
-		(end 168.19049 90.94947)
-		(width 0.254)
-		(layer "B.Cu")
-		(net "NetQ2_1")
-	)
-	(segment
 		(start 174.91749 84.37247)
 		(end 172.86349 84.37247)
@@
 	)
 	(segment
-		(start 167.65544 94.48452)
-		(end 168.94049 93.19947)
-		(width 0.2)
-		(layer "B.Cu")
-		(net "NetQ2_1")
-	)
-	(segment
-		(start 165.68314 94.460255)
-		(end 165.68314 94.48452)
-		(width 0.254)
-		(layer "B.Cu")
-		(net "NetQ2_1")
-	)
-	(segment
 		(start 168.19049 89.04547)
 		(end 168.19049 87.94947)
@@
 		(width 0.254)
 		(layer "B.Cu")
-		(net "NetQ2_1")
-	)
-	(segment
-		(start 168.94049 93.19947)
-		(end 168.19049 92.44947)
-		(width 0.254)
-		(layer "B.Cu")

Commit message: Update BoBa.kicad_pcb
Routing:
- net Vmppt: vias 1 -> 0
Changed lines of the file:
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@@
 		(net "3v3_Primary")
-	)
-	(via
-		(at 141.3491 133.85366)
-		(size 1.27)
-		(drill 0.7112)
-		(layers "F.Cu" "B.Cu")
-		(net "Vmppt")
 	)
 	(segment
