File: BoBa/BoBa.kicad_pcb (KiCad board)
At the start: 4 copper layers, 90.3 x 95.8 mm, 41 parts, among them J1 DF13C-2P-1.25V(21), J2 DF13C-2P-1.25V(21), J3 DF13C-2P-1.25V(21), J4 DF13C-2P-1.25V(21), Q1 FQD13N06LTM, Q2 FQD13N06LTM, U1 LTC4231HUD-2#TRPBF, U2 INA219, U3 INA219AIDCNR, U4_IN-A LTC4231IUD-2#TRPBF, U5 INA219AIDCNR

Commit message: Changed footprint assignemnts and reduced warnings. 10 left.
Parts:
- R7, RS1, RS2: footprint PE1206DRM470R025L:RESC3216X89N -> Vault:RESC3216X89N
Changed lines of the file:
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@@
 		)
 	)
-	(footprint "PE1206DRM470R025L:RESC3216X89N"
+	(footprint "Vault:RESC3216X89N"
 		(layer "B.Cu")
 		(at 129.66978 94.76796 90)
 		(property "Reference" "R7"
-			(at -0.18151 2.02071 270)
+			(at -0.376995 -2.092585 270)
 			(unlocked yes)
 			(layer "B.SilkS")
 			(effects
 				(font
-					(size 1 1)
+					(size 1 0.8128)
 					(thickness 0.15)
+					(bold yes)
 				)
 				(justify mirror)
@@
 		)
 		(property "Value" "PE1206DRM470R025L1"
-			(at 11.23527 -2.784602 270)
+			(at 10.727435 -2.784602 90)
 			(unlocked yes)
 			(layer "B.SilkS")
@@
 		)
 		(property "Datasheet" ""
-			(at 0 0 90)
+			(at 0 0 270)
 			(layer "F.Fab")
 			(hide yes)
@@
 		)
 		(property "Description" ""
-			(at 0 0 90)
+			(at 0 0 270)
 			(layer "F.Fab")
 			(hide yes)
@@
 		)
 		(fp_line
-			(start -0.55 0.93001)
-			(end 0.55 0.93001)
+			(start -0.55 0.93)
+			(end 0.55 0.93)
 			(stroke
 				(width 0.127)
@@
 		(fp_line
 			(start 2.331 -1.181)
-			(end 2.331 1.18101)
+			(end 2.331 1.181)
 			(stroke
 				(width 0.05)
@@
 		(fp_line
 			(start -2.331 -1.181)
-			(end -2.331 1.18101)
+			(end -2.331 1.181)
 			(stroke
 				(width 0.05)
@@
 		)
 		(fp_line
-			(start -2.331 1.18101)
-			(end 2.331 1.18101)
+			(start -2.331 1.181)
+			(end 2.331 1.181)
 			(stroke
 				(width 0.05)
@@
 		(fp_line
 			(start 1.73 -0.93)
-			(end 1.73 0.93001)
+			(end 1.73 0.93)
 			(stroke
 				(width 0.127)
@@
 		(fp_line
 			(start -1.73 -0.93)
-			(end -1.73 0.93001)
+			(end -1.73 0.93)
 			(stroke
 				(width 0.127)
@@
 		)
 		(fp_line
-			(start -1.73 0.93001)
-			(end 1.73 0.93001)
+			(start -1.73 0.93)
+			(end 1.73 0.93)
 			(stroke
 				(width 0.127)
@@
 		)
 		(pad "1" smd rect
-			(at -1.476 0 90)
+			(at -1.476 0 270)
 			(size 1.21 1.86)
 			(layers "B.Cu" "B.Mask" "B.Paste")
@@
 		)
 		(pad "2" smd rect
-			(at 1.476 0 90)
+			(at 1.476 0 270)
 			(size 1.21 1.86)
 			(layers "B.Cu" "B.Mask" "B.Paste")
@@
 		(embedded_fonts no)
 	)
-	(footprint "PE1206DRM470R025L:RESC3216X89N"
+	(footprint "Vault:RESC3216X89N"
 		(layer "B.Cu")
 		(at 165.34944 100.29059 180)
 		(property "Reference" "RS1"
-			(at -3.84105 0.34112 0)
+			(at 1.15895 -4.65888 0)
 			(unlocked yes)
 			(layer "B.SilkS")
@@
 					(size 1 1)
 					(thickness 0.15)
+					(bold yes)
 				)
 				(justify mirror)
@@
 		)
 		(property "Value" "PE1206DRM470R025L"
-			(at 10.727435 -2.784602 0)
+			(at 10.727435 -2.784602 180)
 			(unlocked yes)
 			(layer "B.SilkS")
@@
 		)
 		(property "Datasheet" ""
-			(at 0 0 180)
+			(at 0 0 0)
 			(layer "F.Fab")
 			(hide yes)
@@
 		)
 		(property "Description" ""
-			(at 0 0 180)
+			(at 0 0 0)
 			(layer "F.Fab")
 			(hide yes)
@@
 		(duplicate_pad_numbers_are_jumpers no)
 		(fp_line
-			(start 0.55 0.93)
-			(end -0.55 0.93)
+			(start -0.55 0.93)
+			(end 0.55 0.93)
 			(stroke
 				(width 0.127)
@@
 		)
 		(fp_line
-			(start 0.55 -0.93)
-			(end -0.55 -0.93)
+			(start -0.55 -0.93)
+			(end 0.55 -0.93)
 			(stroke
 				(width 0.127)
@@
 			)
 			(layer "B.SilkS")
-		)
-		(fp_line
-			(start 2.331 1.181)
-			(end -2.331 1.181)
-			(stroke
-				(width 0.05)
-				(type solid)
-			)
-			(layer "B.CrtYd")
 		)
 		(fp_line
@@
 		)
 		(fp_line
-			(start 2.331 -1.181)
-			(end -2.331 -1.181)
+			(start -2.331 1.181)
+			(end 2.331 1.181)
+			(stroke
+				(width 0.05)
+				(type solid)
+			)
+			(layer "B.CrtYd")
+		)
+		(fp_line
+			(start -2.331 -1.181)
+			(end 2.331 -1.181)
 			(stroke
 				(width 0.05)
@@
 		)
 		(fp_line
-			(start 1.73 0.93)
-			(end -1.73 0.93)
-			(stroke
-				(width 0.127)
-				(type solid)
-			)
-			(layer "B.Fab")
-		)
-		(fp_line
 			(start 1.73 -0.93)
 			(end 1.73 0.93)
@@
 		)
 		(fp_line
-			(start 1.73 -0.93)
-			(end -1.73 -0.93)
+			(start -1.73 0.93)
+			(end 1.73 0.93)
+			(stroke
+				(width 0.127)
+				(type solid)
+			)
+			(layer "B.Fab")
+		)
+		(fp_line
+			(start -1.73 -0.93)
+			(end 1.73 -0.93)
 			(stroke
 				(width 0.127)
@@
 		)
 		(pad "1" smd rect
-			(at -1.476 0 180)
+			(at -1.476 0)
 			(size 1.21 1.86)
 			(layers "B.Cu" "B.Mask" "B.Paste")
@@
 		)
 		(pad "2" smd rect
-			(at 1.476 0 180)
+			(at 1.476 0)
 			(size 1.21 1.86)
 			(layers "B.Cu" "B.Mask" "B.Paste")
@@
 		(model "kicad-embed://step_temp_3.STEP"
 			(offset
-				(xyz -0 -0 0)
+				(xyz -0 0 0)
 			)
 			(scale
@@
 		)
 	)
-	(footprint "PE1206DRM470R025L:RESC3216X89N"
+	(footprint "Vault:RESC3216X89N"
 		(layer "B.Cu")
 		(at 121.28359 89.54392 90)
 		(property "Reference" "RS2"
-			(at -0.376995 -2.092585 90)
+			(at -0.376995 -2.092585 270)
 			(unlocked yes)
 			(layer "B.SilkS")
@@
 		)
 		(property "Value" "PE1206DRM470R025L"
-			(at 10.727435 -2.784602 270)
+			(at 10.727435 -2.784602 90)
 			(unlocked yes)
 			(layer "B.SilkS")
@@
 		)
 		(property "Datasheet" ""
-			(at 0 0 90)
+			(at 0 0 270)
 			(layer "F.Fab")
 			(hide yes)
@@
 		)
 		(property "Description" ""
-			(at 0 0 90)
+			(at 0 0 270)
 			(layer "F.Fab")
 			(hide yes)
@@
 		)
 		(pad "1" smd rect
-			(at -1.476 0 90)
+			(at -1.476 0 270)
 			(size 1.21 1.86)
 			(layers "B.Cu" "B.Mask" "B.Paste")
@@
 		)
 		(pad "2" smd rect
-			(at 1.476 0 90)
+			(at 1.476 0 270)
 			(size 1.21 1.86)
 			(layers "B.Cu" "B.Mask" "B.Paste")
