File: BoBa/BoBa.kicad_sch (KiCad schematic)
At the start: 24 parts, among them Q7 FQD13N06LTM, Q8 FQD13N06LTM, U25 INA219, U26 INA219AIDCNR, U27 INA219AIDCNR, U28 LTC4231HUD-2#TRPBF

Commit message: Configure Vault footprint library and reduce DRC warnings from 92 -> 66
Parts:
- C4: footprint FP-GRM155-0_05-IPC_B -> Vault:FP-GRM155-0_05-IPC_B
- FB13, FB14, FB15, FB16: footprint FP-BLM15-0_05-IPC_B -> Vault:FP-BLM15-0_05-IPC_B
- Q7: footprint FAIR-TO-252-3_V -> Vault:FAIR-TO-252-3_V
- Q8: footprint C__Users_Public_Documents_SnapEDA Altium Plugin_libraries_SnapEDA_Library_FQD13N06LTM.PcbLib:TO229P991X239-3N -> Vault:TO229P991X239-3N
- R42, RS7, RS8: footprint C__Users_Public_Documents_SnapEDA Altium Plugin_libraries_SnapEDA_Library_PE1206DRM470R025L.PcbLib:RESC3216X89N -> Vault:RESC3216X89N
- R43, R44, R45, R46: footprint RESC3116X70X50ML13T20 -> Vault:RESC3116X70X50ML13T20
- R47: footprint RESC3225X60N -> Vault:RESC3225X60N
- R48: footprint FP-RG1005-MFG -> Vault:FP-RG1005-MFG
- R49: footprint FP-RG1005-IPC_B -> Vault:FP-RG1005-IPC_B
- R50: footprint CAPC1005X06N -> Vault:CAPC1005X06N
- R51: footprint FP-ERJ2RK-MFG -> Vault:FP-ERJ2RK-MFG
- U25: footprint SOT23-8 -> Vault:SOT23-8
- U26, U27: footprint FP-DCN0008A-IPC_B -> Vault:FP-DCN0008A-IPC_B
- U28: footprint FP-UD-12-05-08-1855-IPC_B -> Vault:FP-UD-12-05-08-1855-IPC_B
Changed lines of the file:
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@@
 			)
 		)
-		(property "Footprint" "FP-BLM15-0_05-IPC_B"
+		(property "Footprint" "Vault:FP-BLM15-0_05-IPC_B"
 			(at 128.27 254 0)
 			(hide yes)
@@
 			)
 		)
-		(property "Footprint" "RESC3116X70X50ML13T20"
+		(property "Footprint" "Vault:RESC3116X70X50ML13T20"
 			(at 146.05 231.14 0)
 			(hide yes)
@@
 			)
 		)
-		(property "Footprint" "FP-BLM15-0_05-IPC_B"
+		(property "Footprint" "Vault:FP-BLM15-0_05-IPC_B"
 			(at 128.27 231.14 0)
 			(hide yes)
@@
 			)
 		)
-		(property "Footprint" "C__Users_Public_Documents_SnapEDA Altium Plugin_libraries_SnapEDA_Library_PE1206DRM470R025L.PcbLib:RESC3216X89N"
+		(property "Footprint" "Vault:RESC3216X89N"
 			(at 77.47 124.46 0)
 			(hide yes)
@@
 			)
 		)
-		(property "Footprint" "FAIR-TO-252-3_V"
+		(property "Footprint" "Vault:FAIR-TO-252-3_V"
 			(at 273.05 45.72 0)
 			(hide yes)
@@
 			)
 		)
-		(property "Footprint" "FP-GRM155-0_05-IPC_B"
+		(property "Footprint" "Vault:FP-GRM155-0_05-IPC_B"
 			(at 361.95 137.16 0)
 			(hide yes)
@@
 			)
 		)
-		(property "Footprint" "RESC3116X70X50ML13T20"
+		(property "Footprint" "Vault:RESC3116X70X50ML13T20"
 			(at 146.05 246.38 0)
 			(hide yes)
@@
 			)
 		)
-		(property "Footprint" "SOT23-8"
+		(property "Footprint" "Vault:SOT23-8"
 			(at 74.93 104.14 0)
 			(hide yes)
@@
 			)
 		)
-		(property "Footprint" "C__Users_Public_Documents_SnapEDA Altium Plugin_libraries_SnapEDA_Library_PE1206DRM470R025L.PcbLib:RESC3216X89N"
+		(property "Footprint" "Vault:RESC3216X89N"
 			(at 303.53 83.82 0)
 			(hide yes)
@@
 			)
 		)
-		(property "Footprint" "RESC3116X70X50ML13T20"
+		(property "Footprint" "Vault:RESC3116X70X50ML13T20"
 			(at 146.05 238.76 0)
 			(hide yes)
@@
 			)
 		)
-		(property "Footprint" "FP-DCN0008A-IPC_B"
+		(property "Footprint" "Vault:FP-DCN0008A-IPC_B"
 			(at 161.29 154.94 0)
 			(hide yes)
@@
 			)
 		)
-		(property "Footprint" "FP-BLM15-0_05-IPC_B"
+		(property "Footprint" "Vault:FP-BLM15-0_05-IPC_B"
 			(at 128.27 238.76 0)
 			(hide yes)
@@
 			)
 		)
-		(property "Footprint" "FP-RG1005-MFG"
+		(property "Footprint" "Vault:FP-RG1005-MFG"
 			(at 285.75 101.6 0)
 			(hide yes)
@@
 			)
 		)
-		(property "Footprint" "RESC3225X60N"
+		(property "Footprint" "Vault:RESC3225X60N"
 			(at 285.75 91.44 0)
 			(hide yes)
@@
 			)
 		)
-		(property "Footprint" "FP-DCN0008A-IPC_B"
+		(property "Footprint" "Vault:FP-DCN0008A-IPC_B"
 			(at 293.37 38.1 0)
 			(hide yes)
@@
 			)
 		)
-		(property "Footprint" "C__Users_Public_Documents_SnapEDA Altium Plugin_libraries_SnapEDA_Library_PE1206DRM470R025L.PcbLib:RESC3216X89N"
+		(property "Footprint" "Vault:RESC3216X89N"
 			(at 130.81 177.8 0)
 			(hide yes)
@@
 			)
 		)
-		(property "Footprint" "FP-RG1005-IPC_B"
+		(property "Footprint" "Vault:FP-RG1005-IPC_B"
 			(at 285.75 119.38 0)
 			(hide yes)
@@
 			)
 		)
-		(property "Footprint" "C__Users_Public_Documents_SnapEDA Altium Plugin_libraries_SnapEDA_Library_FQD13N06LTM.PcbLib:TO229P991X239-3N"
+		(property "Footprint" "Vault:TO229P991X239-3N"
 			(at 346.71 60.96 0)
 			(hide yes)
@@
 			)
 		)
-		(property "Footprint" "FP-BLM15-0_05-IPC_B"
+		(property "Footprint" "Vault:FP-BLM15-0_05-IPC_B"
 			(at 128.27 246.38 0)
 			(hide yes)
@@
 			)
 		)
-		(property "Footprint" "CAPC1005X06N"
+		(property "Footprint" "Vault:CAPC1005X06N"
 			(at 285.75 137.16 0)
 			(hide yes)
@@
 			)
 		)
-		(property "Footprint" "FP-ERJ2RK-MFG"
+		(property "Footprint" "Vault:FP-ERJ2RK-MFG"
 			(at 349.25 68.58 0)
 			(hide yes)
@@
 			)
 		)
-		(property "Footprint" "RESC3116X70X50ML13T20"
+		(property "Footprint" "Vault:RESC3116X70X50ML13T20"
 			(at 146.05 254 0)
 			(hide yes)
@@
 			)
 		)
-		(property "Footprint" "FP-UD-12-05-08-1855-IPC_B"
+		(property "Footprint" "Vault:FP-UD-12-05-08-1855-IPC_B"
 			(at 295.91 101.6 0)
 			(hide yes)
