File: BoBa/INA.kicad_sch (KiCad schematic)
At the start: 4 parts, among them U20 LTC4231IUD-2#TRPBF

Commit message: Configure Vault footprint library and reduce DRC warnings from 92 -> 66
Parts:
- C16: footprint FP-GRM155-0_05-IPC_B -> Vault:FP-GRM155-0_05-IPC_B
- IN-A1: renamed from IN-A; footprint INF-PG-SOT23_M -> Vault:INF-PG-SOT23_M
- R31: footprint FP-ERJ2RK-MFG -> Vault:FP-ERJ2RK-MFG
- U20: footprint FP-UD-12-05-08-1855-IPC_A -> Vault:FP-UD-12-05-08-1855-IPC_A
Changed lines of the file:
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@@
 			)
 		)
-		(property "Footprint" "FP-ERJ2RK-MFG"
+		(property "Footprint" "Vault:FP-ERJ2RK-MFG"
 			(at 133.35 36.83 0)
 			(hide yes)
@@
 		)
 		(instances
-			(project "BoBa"
-				(path "/eea5ac2b-0263-4b76-a86f-96656803f600/59f67bea-5f0a-4bcd-8759-a7c2fd72ecbb"
-					(reference "R30")
-					(unit 1)
-				)
-			)
 			(project "BoBa"
 				(path "/ffd05940-f180-4d71-86aa-98b5fd06b3da/b3ff1496-97f2-4268-bcc9-3f742454327d"
@@
 		(instances
 			(project "BoBa"
-				(path "/eea5ac2b-0263-4b76-a86f-96656803f600/59f67bea-5f0a-4bcd-8759-a7c2fd72ecbb"
-					(reference "#PWR047")
-					(unit 1)
-				)
-			)
-			(project "BoBa"
 				(path "/ffd05940-f180-4d71-86aa-98b5fd06b3da/b3ff1496-97f2-4268-bcc9-3f742454327d"
 					(reference "#PWR048")
@@
 		(instances
 			(project "BoBa"
-				(path "/eea5ac2b-0263-4b76-a86f-96656803f600/59f67bea-5f0a-4bcd-8759-a7c2fd72ecbb"
-					(reference "#PWR038")
-					(unit 1)
-				)
-			)
-			(project "BoBa"
 				(path "/ffd05940-f180-4d71-86aa-98b5fd06b3da/b3ff1496-97f2-4268-bcc9-3f742454327d"
 					(reference "#PWR039")
@@
 		(in_pos_files yes)
 		(dnp no)
-		(property "Reference" "IN-A"
+		(property "Reference" "IN-A1"
 			(at 130.556 20.574 0)
 			(show_name no)
@@
 			)
 		)
-		(property "Footprint" "INF-PG-SOT23_M"
+		(property "Footprint" "Vault:INF-PG-SOT23_M"
 			(at 130.81 29.21 0)
 			(hide yes)
@@
 		(instances
 			(project "BoBa"
-				(path "/eea5ac2b-0263-4b76-a86f-96656803f600/59f67bea-5f0a-4bcd-8759-a7c2fd72ecbb"
-					(reference "1114211111")
-					(unit 1)
-				)
-			)
-			(project "BoBa"
 				(path "/ffd05940-f180-4d71-86aa-98b5fd06b3da/b3ff1496-97f2-4268-bcc9-3f742454327d"
-					(reference "IN-A")
+					(reference "IN-A1")
 					(unit 1)
 				)
@@
 			)
 		)
-		(property "Footprint" "FP-UD-12-05-08-1855-IPC_A"
+		(property "Footprint" "Vault:FP-UD-12-05-08-1855-IPC_A"
 			(at 85.09 54.61 0)
 			(hide yes)
@@
 		)
 		(instances
-			(project "BoBa"
-				(path "/eea5ac2b-0263-4b76-a86f-96656803f600/59f67bea-5f0a-4bcd-8759-a7c2fd72ecbb"
-					(reference "U19")
-					(unit 1)
-				)
-			)
 			(project "BoBa"
 				(path "/ffd05940-f180-4d71-86aa-98b5fd06b3da/b3ff1496-97f2-4268-bcc9-3f742454327d"
@@
 			)
 		)
-		(property "Footprint" "FP-GRM155-0_05-IPC_B"
+		(property "Footprint" "Vault:FP-GRM155-0_05-IPC_B"
 			(at 146.05 74.93 0)
 			(hide yes)
@@
 		)
 		(instances
-			(project "BoBa"
-				(path "/eea5ac2b-0263-4b76-a86f-96656803f600/59f67bea-5f0a-4bcd-8759-a7c2fd72ecbb"
-					(reference "C15")
-					(unit 1)
-				)
-			)
 			(project "BoBa"
 				(path "/ffd05940-f180-4d71-86aa-98b5fd06b3da/b3ff1496-97f2-4268-bcc9-3f742454327d"
@@
 		(instances
 			(project "BoBa"
-				(path "/eea5ac2b-0263-4b76-a86f-96656803f600/59f67bea-5f0a-4bcd-8759-a7c2fd72ecbb"
-					(reference "#PWR041")
-					(unit 1)
-				)
-			)
-			(project "BoBa"
 				(path "/ffd05940-f180-4d71-86aa-98b5fd06b3da/b3ff1496-97f2-4268-bcc9-3f742454327d"
