File: PoBoI/3V3Secondary.kicad_sch (KiCad schematic)
At the start: 17 parts, among them Q1 SI7164DP-T1-GE3, Q4 SI5418DU-T1-GE3, U12 INA219AIDCNR, U15 LTC4231IUD-2#TRPBF

Commit message: POBOI 4S updates: remove 12V/TVS sheets, fix VBATT dividers, INA219 addresses, U26
POBOI changes 10/28 Simon Ionashku

- Deleted the separate copy of the PCB file (BoardFix, it was an older version)
- Removed these sheets from the schematic and the board (no use for them anymore)
   - 12 PRIMARY
   - 12V BOOST
   - 12V SECONDARY
      - our 4S pack is already 12-16.8V so boosting to 12V does nothing, and the LM2622 is only rated for 12V in anyway
      - anything that needs ~12V can just use the VBATT Primary/Secondary rails
      - also deleted the "NEED TO ADD 12V COMPATIBILITY" note on the STM32 sheet
   - TVS_DIODES
      - they weren't actually connected to anything (cathodes were all no-connects)
      - they're also just 3.6V zeners, not real TVS diodes
      - the LTC4231 already shuts off on overvoltage, undervoltage and overcurrent, and there's a small zener clamp on each enable line
- Fixed the VBATT Primary and Secondary divider resistors since they were still using the 2S numbers and we moved to 4S
   - with the old values the switches would've never turned on (they cut off above ~8V)
   - new thresholds: OVoff = 17.5V, UVon = 12.4V, UVoff = 12.0V (3.0V per cell)
   - RES    OLD     NEW
      R71    866k    931k   (Primary)
      R74    2.37k   2.15k  (Primary)
      R77    37.4k   18.7k  (Primary)
      R78    100k    45.3k  (Primary)
      R68    866k    931k   (Secondary)
      R65    2.37k   2.15k  (Secondary)
      R63    37.4k   18.7k  (Secondary)
      R64    100k    45.3k  (Secondary)
   - updated the values, part numbers and form factor (all 0603 now) in the BOM and field table
      - R68/R71 were 0201 rated for 25V which is cutting it close at 16.8V
   - updated the notes and calculations on both sheets
- Fixed the INA219 addresses
   - a bunch of the A0/A1 pins were floating (marked no-connect) so the addresses would've been random
   - went through and checked/corrected all six so A0 and A1 match the slave address table
      5V Primary    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
Parts:
- R13, R14: now not fitted
Connections:
- net SCL: now also U12.7 (A0)
- no-connect marks 1 -> 0
