File: PoBoI/LEARNSAT_POBOY_v3.2.0.kicad_pcb (KiCad board)
At the start: 4 copper layers, 90.2 x 95.8 mm, 489 parts, among them J1 FTSH-105-01-L-DV-K-P-TR, J5 FTSH-105-01-L-DV-K-P-TR, P1 22-28-4036, Q1 SI7164DP-T1-GE3, Q10 SI5418DU-T1-GE3, Q11 SI7164DP-T1-GE3, Q12 SI5418DU-T1-GE3, Q13 SI5418DU-T1-GE3, Q13 SI7164DP-T1-GE3, Q14 SI5418DU-T1-GE3, Q14 SI7164DP-T1-GE3, Q15 SI7164DP-T1-GE3, Q16 SI5418DU-T1-GE3, Q17 SI7164DP-T1-GE3, Q18 SI5418DU-T1-GE3, Q19 SI7164DP-T1-GE3, Q2 SI7164DP-T1-GE3, Q20 SI5418DU-T1-GE3, Q20 SI7164DP-T1-GE3, Q21 SI7164DP-T1-GE3, Q22 SI5418DU-T1-GE3, Q23 SI7164DP-T1-GE3, Q24 SI5418DU-T1-GE3, Q3 SI7164DP-T1-GE3, Q4 SI5418DU-T1-GE3, Q5 SI5418DU-T1-GE3, Q6 SI7164DP-T1-GE3, Q7 SI7164DP-T1-GE3, Q8 SI5418DU-T1-GE3, Q9 SI5418DU-T1-GE3, SW1 B3U-1000P, SW2 B3U-1000P, SW3 TS04-66-43-BK-100-SMT, U1 MAX6746KA29+T, U1 STM32F103RET6, U10 LM2622MMX-ADJ/NOPB, U11 LM2622MMX-ADJ/NOPB, U12 INA219AIDCNR, U13 INA219AIDCNR, U14 INA219AIDCNR, U15 LTC4231IUD-2#TRPBF, U16 LTC4231IUD-2#TRPBF, U17 LP5907SNX-3.3, U18 LP5907SNX-3.3, U18 LTC4231IUD-2#TRPBF, U19 INA219AIDCNR, U2 SN74AUP1G08QDCKRQ1, U20 INA219AIDCNR, U21 74AC14MTCX, U22 LTC4231IUD-2#TRPBF, U22 LTC4304CMS#PBF, U23 INA219AIDCNR, U23 SN74LVC1G373DCKR, U24 LTC4231IUD-2#TRPBF, U25 INA219AIDCNR, U25 LTC4231IUD-2#TRPBF, U26 ISL3259EIRZ, U26 LTC4231IUD-2#TRPBF, U27 INA219AIDCNR, U28 LTC4231IUD-2#TRPBF, U29 INA219AIDCNR, U29 LTC4231IUD-2#TRPBF, U3 MAX6746KA29+T, U30 INA219AIDCNR, U30 LTC4231IUD-2#TRPBF, U31 INA219AIDCNR, U32 LTC4231IUD-2#TRPBF, U33 INA219AIDCNR, U34 MAX6746KA29+T, U35 MAX6746KA29+T, U36 SN74AUP1G08QDCKRQ1, U37 SN74AUP1G08QDCKRQ1, U38 LTC4304CMS#PBF, U39 74AC14MTCX, U4 SN74AUP1G08QDCKRQ1, U40 SN74LVC1G373DCKR, U41 ISL3259EIRZ, U5 LT1616ES6#TRMPBF, U50 LM2622MMX-ADJ/NOPB, U51 LM2622MMX-ADJ/NOPB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

Commit message: POBOI 4S updates: remove 12V/TVS sheets, fix VBATT dividers, INA219 addresses, U26
POBOI changes 10/28 Simon Ionashku

- Deleted the separate copy of the PCB file (BoardFix, it was an older version)
- Removed these sheets from the schematic and the board (no use for them anymore)
   - 12 PRIMARY
   - 12V BOOST
   - 12V SECONDARY
      - our 4S pack is already 12-16.8V so boosting to 12V does nothing, and the LM2622 is only rated for 12V in anyway
      - anything that needs ~12V can just use the VBATT Primary/Secondary rails
      - also deleted the "NEED TO ADD 12V COMPATIBILITY" note on the STM32 sheet
   - TVS_DIODES
      - they weren't actually connected to anything (cathodes were all no-connects)
      - they're also just 3.6V zeners, not real TVS diodes
      - the LTC4231 already shuts off on overvoltage, undervoltage and overcurrent, and there's a small zener clamp on each enable line
- Fixed the VBATT Primary and Secondary divider resistors since they were still using the 2S numbers and we moved to 4S
   - with the old values the switches would've never turned on (they cut off above ~8V)
   - new thresholds: OVoff = 17.5V, UVon = 12.4V, UVoff = 12.0V (3.0V per cell)
   - RES    OLD     NEW
      R71    866k    931k   (Primary)
      R74    2.37k   2.15k  (Primary)
      R77    37.4k   18.7k  (Primary)
      R78    100k    45.3k  (Primary)
      R68    866k    931k   (Secondary)
      R65    2.37k   2.15k  (Secondary)
      R63    37.4k   18.7k  (Secondary)
      R64    100k    45.3k  (Secondary)
   - updated the values, part numbers and form factor (all 0603 now) in the BOM and field table
      - R68/R71 were 0201 rated for 25V which is cutting it close at 16.8V
   - updated the notes and calculations on both sheets
- Fixed the INA219 addresses
   - a bunch of the A0/A1 pins were floating (marked no-connect) so the addresses would've been random
   - went through and checked/corrected all six so A0 and A1 match the slave address table
      5V Primary    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
Parts:
- removed C102: 0.1uF, Vault:FP-C0603-CJ-MFG
- removed C103, C104: GRM0335C1E100JA01D, Vault:FP-GRM033-0_03-IPC_A
- removed C120, C28: Capacitor 1 uF +/- 10% 25 V 0603, Vault:CAPC1608X90X40LL10T20
- removed C121, C34: Capacitor 1uF +/- 10% 16V 0603, Vault:CAPC1608X90X35ML15T15
- removed C122, C33: C0805C184K5RACTU, Vault:FP-C0805C-DN-IPC_A
- removed C99: Capacitor 1 uF +/- 10% 16 V 0603, Vault:CAPC1608X94X35NL15T15
- removed the Cc1 at (241.9, 166.3)
- removed Cc2: 2.2nF, Vault:FP-C0402-BB-MFG
- removed the Cin1 at (239.9, 170.7)
- removed Cin2, Cout2: 22uF, Vault:FP-CL31-IPC_A
- removed the Cout1 at (236.4, 161.7)
- removed D19, D20: 1N914BWT, Vault:FP-502-01-MFG
- removed D23, D38, D41, D47, D50, D?: MM3Z3V6T1G, Vault:ONSC-SOD-323-2-477-02_V
- removed D63, D64: 1N4148WX-TP, Vault:1N4148WX-TP-Footprint-1
- removed the D8 at (545.0, 168.7)
- removed the H1 at (345.5, 64.4)
- removed the H2 at (345.5, 59.3)
- removed J5: FTSH-105-01-L-DV-K-P-TR, Vault:FP-FTSH-105-01-L-DV-K-P-T-MFG
- removed the L3 at (339.8, 120.6)
- removed L5, L6: 10uH, Vault:FP-MLZ1608-IPC_C
- removed the P1 at (338.6, 64.2)
- removed Q12, Q?: SI5418DU-T1-GE3, Vault:SI5418DU-T1-GE3-Footprint-1
- removed the Q20 at (440.6, 135.9)
- removed Q3: SI7164DP-T1-GE3, Vault:Vishay_S17-0173-SINGLE_MFG
- removed R15, R157, R158, R16: CRCW12103K30JNEA, Vault:FP-CRCW1210-e3-IPC_C
- removed R150, R28: CSR1206FK25L0, Vault:FP-CSR1206-IPC_C
- removed R151, R37: 768KR2F, Vault:RESC0402(1005)_L
- removed R152, R35: CRCW12067K50FKEA, Vault:FP-CRCW1206-e3-IPC_A
- removed R153, R39: PTN0603E8002BST1, Vault:FP-PTN0603-IPC_B
- removed R154: RT1206FRE07150KL, Vault:FP-RT1206-IPC_C
- removed R155, R156, R23, R25: Resistor 10R +/-1 % 0402 63 mW, Vault:RESC0402(1005)_L
- removed the R40 at (221.0, 92.4)
- removed the RFB1 at (237.3, 164.2)
- removed the RFB2 at (239.2, 166.2)
- removed RFB3: 7.5kOhms, Vault:FP-ERJ3EK-MFG
- removed RFB4: 64.9kOhms, Vault:RESC3216X70X50NL05T20
- removed the Rc1 at (236.4, 166.2)
- removed Rc2: 24kOhms, Vault:RESC1005X40X25ML05T05
- removed the SW3 at (409.4, 71.6)
- removed U10, U11: LM2622MMX-ADJ/NOPB, Vault:DGK0008A_M
- removed U13, U61: INA219AIDCNR, Vault:FP-DCN0008A-IPC_A
- removed U18, U60: LTC4231IUD-2#TRPBF, Vault:FP-UD-12-05-08-1855-IPC_A
- removed U18: LP5907SNX-3.3, Vault:TI-DQN4-480X480TP_V
- removed U38: LTC4304CMS#PBF, Vault:LTC4304CMS#PBF-Footprint-1
- removed U41: ISL3259EIRZ, Vault:ISL3259EIRZ-Footprint-1
- removed the U7 at (522.7, 171.2)
- removed the U8 at (378.8, 70.1)
- removed the Y1 at (497.0, 59.0)
- R63, R77: value CR0603-FX-3742ELF -> RC0603FR-0718K7L
- R64, R78: value Resistor 100k +/-1% 0402 100 mW -> RC0603FR-0745K3L; footprint Vault:RESC1005X40X25ML05T05 -> Vault:RESC0603(1608)_L
- R65, R74: value 2D37KR2F -> RC0603FR-072K15L; footprint Vault:RESC0402(1005)_L -> Vault:RESC0603(1608)_L
- R68, R71: value MC0201L6F8663SE -> RC0603FR-07931KL; footprint Vault:RESC0603X26X15NL03T05 -> Vault:RESC0603(1608)_L
- U26: value ISL3259EIRZ -> ISL3259EIBZ; footprint Vault:ISL3259EIRZ-Footprint-1 -> Package_SO:SOIC-8_3.9x4.9mm_P1.27mm
- moved SW3 267.9 mm to (409.4, 71.6), turned to 180 degrees
- moved LED1 239.9 mm to (359.0, 36.1)
- moved LED2 239.9 mm to (359.0, 39.2)
- moved LED3 239.9 mm to (359.0, 42.3)
- moved LED4 239.9 mm to (359.0, 45.4)
- moved LED5 239.9 mm to (359.0, 48.5)
- moved LED6 239.9 mm to (359.0, 51.6)
- moved RLED2 222.3 mm to (379.1, 47.0)
- moved RLED3 222.3 mm to (375.1, 47.3)
- moved RLED5 222.3 mm to (379.1, 49.6)
- moved RLED6 222.3 mm to (375.1, 50.3)
- moved RLED1 222.3 mm to (370.9, 47.3)
- moved RLED4 222.3 mm to (370.9, 50.3)
- moved U25 220.4 mm to (434.9, 131.8)
- moved H1 219.9 mm to (345.5, 64.4)
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Connections:
- R60 pad 1: /STM32/RS-485B -> /STM32/RS-485A
- R60 pad 2: /STM32/RS-485A -> /STM32/RS-485B
- U12 pad 7: unconnected-(U12-A0-Pad7) -> SCL
- U14 pad 7: unconnected-(U14-A0-Pad7) -> SDA
- U19 pad 7: unconnected-(U19-A0-Pad7) -> 3V3
- U26 pad 5: 5V_Secondary -> GND
- U26 pad 6: GND -> /STM32/RS-485A
- U26 pad 7: /STM32/RS-485A -> /STM32/RS-485B
- U26 pad 8: /STM32/RS-485B -> 5V_Secondary
- U27 pad 8: unconnected-(U27-A1-Pad8) -> 3V3
- U30 pad 7: unconnected-(U30-A0-Pad7) -> 3V3
- U30 pad 8: unconnected-(U30-A1-Pad8) -> 3V3
Routing:
- net GND: track 274.8 -> 174.6 mm, vias 19 -> 14
- net ???: track 44.4 -> 0.00 mm, vias 2 -> 0
- net Net-(Q12-S_1): track 23.0 -> 0.00 mm, vias 2 -> 0
- net VBatt Primary: track 22.8 -> 0.00 mm
- net 3V3: track 67.9 -> 46.8 mm, vias 4 -> 2
- net Net-(Q3-D): track 20.4 -> 0.00 mm
- net Net-(Q12-G): track 16.7 -> 0.00 mm, vias 2 -> 0
- net 12V: track 14.7 -> 0.00 mm
- net NetQ20_4: track 12.1 -> 0.00 mm
- net NetQ20_5-6-7-8: track 11.6 -> 0.00 mm
- net NetR152_2: track 9.76 -> 0.00 mm
- net NetR151_2: track 9.30 -> 0.00 mm
- net Net-(U13-IN+): track 9.24 -> 0.00 mm
- net NetQ20_1: track 8.97 -> 0.00 mm
- net Net-(U13-IN-): track 8.48 -> 0.00 mm
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- removed copper zone on F.Cu, net BOOST_2
- removed copper zone on F.Cu, net FB_1
- removed copper zone on F.Cu, net FB_2
- removed copper zone on F.Cu, net SW_2
Other:
- board text removed: "12VPrimary"
- board text removed: "12V_Boost"
